File: kicad/vue3/vue3.kicad_sch (KiCad schematic)
At the start: 26 parts, among them J1 Conn_01x07_Male, U5 ESP32-WROVER-IB

Commit message: WIP
Parts:
- removed R143: DNP, symbol Device:R_Small
- removed SP1: Buzzer, symbol Device:Buzzer
- added FD1: Fiducial, symbol Mechanical:Fiducial
- added J29: LPJ4215HENL, Connector_RJ:RJ45_Hanrun_HR911105A_Horizontal, symbol Connector:RJ45_Hanrun_HR911105A_Horizontal
- added MH1: MountingHole, symbol Mechanical:MountingHole
- added U1001: RTL8201F-VB-CG, easyeda2kicad:QFN-32_L5.0-W5.0-P0.50-BL-EP3.4, symbol easyeda2kicad:RTL8201F-VB-CG
- added Y1: 25 Mhz, symbol Device:Crystal
- D3: value LED -> Green
- D31: renamed from D4; value LED -> Blue
- renumbered U5 to M1
Connections:
- net ~{AT_RST} is gone; now on net ETH_LED: M1.26 (IO4)
- net I2CCLK: now also M1.30 (IO18); no longer M1.36 (IO22)
- net I2CDAT: now also M1.29 (IO5); no longer M1.33 (IO21)
- net IO0: now also U1001.15 (TXC)
- net at R115.2, R119.1: no longer M1.7 (IO35)
- net at R114.1, R118.1: no longer M1.6 (IO34)
- net ETH_LED: now reaches R81.1
- net at R113.2, R117.1: no longer M1.9 (IO33)
- net RXD0: now reaches M1.10 (IO25)
- net RXD0: now also U1001.9 (RXD[0])
- net WIFI_LED: now reaches M1.24 (IO2)
- net WIFI_LED: now also R80.2
- net TXD0: now reaches M1.31 (IO19)
- net TXD0: now also U1001.16 (TXD[0])
- net at R112.2, R116.2: no longer M1.8 (IO32)
- net BUZ+: no longer names the net of M1.14 (IO12)
- net BUZ-: no longer names the net of M1.12 (IO27)
- net EMAC_RXD1 renamed RXD1
- net RXD1: now also U1001.10 (RXD[1])
- new net: U1001.31 (CKXTAL1), Y1.1
- new net: U1001.32 (CKXTAL2), Y1.2
- new net MDC: M1.9 (IO33), U1001.22 (MDC)
- new net MDI0+: J29.1 (TD+), U1001.3 (MDI+[0])
- new net MDI0-: J29.4 (TCT), U1001.4 (MDI-[0])
- new net MDI1+: J29.3 (RD+), U1001.5 (MDI+[1])
- new net MDI1-: J29.6 (RD-), U1001.6 (MDI-[1])
- new net MDIO: M1.8 (IO32), U1001.23 (MDIO)
- new net TXD1: M1.36 (IO22), U1001.17 (TXD[1])
Other:
- sheet ADC ports: added none; removed EMAC_RXD1
- moved on the sheet: R43, R44
