File: kicad/vue3/vue3_adc.kicad_sch (KiCad schematic)
At the start: 141 parts, among them J1 AudioJack3_Ground, J10 AudioJack3_Ground, J11 AudioJack3_Ground, J12 AudioJack3_Ground, J13 AudioJack3_Ground, J14 AudioJack3_Ground, J15 AudioJack3_Ground, J16 AudioJack3_Ground, J18 AudioJack3_Ground, J19 AudioJack3_Ground, J2 AudioJack3_Ground, J20 AudioJack3_Ground, J3 AudioJack3_Ground, J5 AudioJack3_Ground, J6 AudioJack3_Ground, J7 AudioJack3_Ground, J8 AudioJack3_Ground, J9 AudioJack3_Ground, U6 ATSAMD09D14A-M, U7 74HC4051, U8 74HC4051

Commit message: WIP
Parts:
- removed C68: DNP, symbol Device:C_Small
- removed H1: Conn_02x05_Odd_Even, symbol Connector_Generic:Conn_02x05_Odd_Even
- removed J1, J10, J11, J12, J13, J14, J15, J16, J18, J19, J2, J20, J3, J5, J6, J7, J8, J9, J?: AudioJack3_Ground, symbol Connector:AudioJack3_Ground
- added J23, J24: Conn_01x08, symbol Connector_Generic:Conn_01x16
- added J26: Conn_01x06, symbol Connector_Generic:Conn_01x06
- R55: tolerance (none) -> 1%
- gave numbers to parts that had none: 1
Connections:
- net +1V8: now also J23.1 (Pin_1), J23.11 (Pin_11), J23.13 (Pin_13), J23.15 (Pin_15), J23.3 (Pin_3), J23.5 (Pin_5), J23.7 (Pin_7), J23.9 (Pin_9), J24.1 (Pin_1), J24.11 (Pin_11), J24.13 (Pin_13), J24.15 (Pin_15), J24.3 (Pin_3), J24.5 (Pin_5), J24.7 (Pin_7), J24.9 (Pin_9), J26.2 (Pin_2), J26.4 (Pin_4), J26.6 (Pin_6)
- net CTE6-: now reaches D14.1 (K), R50.2, R64.1, TPCTE6.1
- net CTE6-: now also J23.6 (Pin_6)
- net CTE5-: now reaches D15.1 (K), R51.1, R65.2, TPCTE5.1
- net CTE5-: now also J23.8 (Pin_8)
- net CTE3-: now reaches D17.1 (K), R53.1, R67.2, TPCTE3.1
- net CTE3-: now also J23.12 (Pin_12)
- net CTE13-: now reaches D29.1 (K), R57.1, R75.2, TPCTE13.1
- net CTE13-: now also J24.8 (Pin_8)
- net CTE4-: now reaches D16.1 (K), R53.1, R67.2, TPCTE4.1
- net CTE4-: now also J23.10 (Pin_10)
- net CTE7-: now reaches D27.1 (K), R88.2, R89.1, TPCTE7.1
- net CTE7-: now also J23.4 (Pin_4)
- net CTE11-: now reaches D19.1 (K), R56.1, R70.2, TPCTE11.1
- net CTE11-: now also J24.12 (Pin_12)
- net CTE12-: now reaches D?.1 (K), R71.2, R76.1, TPCTE12.1
- net CTE12-: now also J24.10 (Pin_10)
- net CTE15-: now reaches D22.1 (K), R59.1, R73.2, TPCTE15.1
- net CTE15-: now also J24.4 (Pin_4)
- net CTE16-: now reaches D23.1 (K), R27.2, R60.1, TPCTE16.1
- net CTE16-: now also J24.2 (Pin_2)
- net CT2-: now reaches D12.1 (K), R48.1, R62.2, TPCT2.1
- net CT2-: now also J26.3 (Pin_3)
- net CTE14-: now reaches D21.1 (K), R58.1, R74.2, TPCTE14.1
- net CTE14-: now also J24.6 (Pin_6)
- net CT1-: now reaches D13.1 (K), R49.1, R63.2, TPCT1.1
- net CT1-: now also J26.1 (Pin_1)
- net CTE1-: now reaches D18.1 (K), R55.1, R69.2, TPCTE1.1
- net CTE1-: now also J23.16 (Pin_16)
- net CTE9-: now reaches D24.1 (K), R94.2, R95.1, TPCTE09.1
- net CTE9-: now also J24.16 (Pin_16)
- net CTE10-: now reaches D25.1 (K), R95.2, R96.1, TPCTE10.1
- net CTE10-: now also J24.14 (Pin_14)
- net CTE8-: now reaches D26.1 (K), R90.2, R91.1, TPCTE8.1
- net CTE8-: now also J23.2 (Pin_2)
- net CT3-: now reaches D11.1 (K), R47.1, R61.2, TPCT3.1
- net CT3-: now also J26.5 (Pin_5)
- net CTE2-: now reaches D28.1 (K), R54.1, R68.2, TPCTE2.1
- net CTE2-: now also J23.14 (Pin_14)
- net S2 renamed ?
- no-connect marks 38 -> 0
Other:
- note added: "L=Black=plus K=White=minus"
- moved on the sheet: C10, C11, C38, C39, C51, C78, C80, C81, C9, R141, R78, R83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
