File: kicad/vue3/vue3_psu.kicad_sch (KiCad schematic)
At the start: 61 parts, among them U1 BGFCN8

Commit message: WIP
Parts:
- removed R1, R3: R, symbol Device:R
- added F1, F2: 4A, symbol Device:R
- added J26: Conn_01x05, symbol Connector_Generic:Conn_01x05
- DA1: value MB6S -> MB6F
- F3: renamed from R5; value R -> 4A
- renumbered TR1 to FL1, R19 to R246, R15 to R247, R17 to R248, TPN1 to TPP1, TPN2 to TPP2, TPN3 to TPP3
Connections:
- net AC: now also F1.2, F2.2, J26.1 (Pin_1), J26.2 (Pin_2), J26.3 (Pin_3), J26.5 (Pin_5)
- net at C67.1, DA1.2, R120.1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: now also F1.1
- net at R136.1, R4.2: now also F2.1
- no-connect marks 0 -> 1
